File: KiCAD/ButtonBar/button_bar.sch (KiCad schematic (older format))
At the start: 14 parts, among them P1 Buttons, SW1 SW_UP, SW2 SW_DN, SW3 SW_OK, SW4 SW_LT, SW5 SW_RT, SW6 RESET

Commit message: button board pcb update ajm
Parts:
- added H1, H2, H3, H4: CONN_1, symbol CONN_1
- renumbered R10 to R6
Connections:
- no-connect marks 0 -> 4
Changed lines of the file:
@@
 $EndComp
 $Comp
-L GND #PWR01
+L GND #PWR1
 U 1 1 5303F82B
 P 1750 6550
-F 0 "#PWR01" H 1750 6550 30  0001 C CNN
+F 0 "#PWR1" H 1750 6550 30  0001 C CNN
 F 1 "GND" H 1750 6480 30  0001 C CNN
 F 2 "" H 1750 6550 60  0000 C CNN
@@
 $EndComp
 $Comp
-L R R10
+L R R6
 U 1 1 5303FB7E
 P 1750 5550
-F 0 "R10" V 1830 5550 40  0000 C CNN
+F 0 "R6" V 1830 5550 40  0000 C CNN
 F 1 "10K" V 1757 5551 40  0000 C CNN
 F 2 "RC03" V 1680 5550 30  0001 C CNN
@@
 $EndComp
 $Comp
-L PWR_FLAG #FLG02
+L PWR_FLAG #FLG1
 U 1 1 5303FDCF
 P 3150 1700
-F 0 "#FLG02" H 3150 1795 30  0001 C CNN
+F 0 "#FLG1" H 3150 1795 30  0001 C CNN
 F 1 "PWR_FLAG" H 3150 1880 30  0000 C CNN
 F 2 "" H 3150 1700 60  0000 C CNN
@@
 $EndComp
 $Comp
-L PWR_FLAG #FLG03
+L PWR_FLAG #FLG2
 U 1 1 5303FDDE
 P 2050 6450
-F 0 "#FLG03" H 2050 6545 30  0001 C CNN
+F 0 "#FLG2" H 2050 6545 30  0001 C CNN
 F 1 "PWR_FLAG" H 2050 6630 30  0000 C CNN
 F 2 "" H 2050 6450 60  0000 C CNN
@@
 	2050 6450 2050 6150
 Connection ~ 2050 6150
-Wire Wire Line
-	5200 4050 4400 4050
 $Comp
 L C C1
@@
 Wire Wire Line
 	4650 3250 4650 3150
-Connection ~ 4850 4050
 Text Label 3875 6150 0    60   ~ 0
 RST
@@
 	5000 3150 5000 3950
 Connection ~ 5000 3950
+Wire Wire Line
+	5200 4050 4400 4050
+$Comp
+L CONN_1 H1
+U 1 1 53077F02
+P 6450 5000
+F 0 "H1" V 6550 4975 40  0000 L CNN
+F 1 "CONN_1" H 6450 5055 30  0001 C CNN
+F 2 "" H 6450 5000 60  0000 C CNN
+F 3 "" H 6450 5000 60  0000 C CNN
+	1    6450 5000
+	0    -1   -1   0
+$EndComp
+$Comp
+L CONN_1 H2
+U 1 1 53077F28
+P 6650 5000
+F 0 "H2" V 6750 4975 40  0000 L CNN
+F 1 "CONN_1" H 6650 5055 30  0001 C CNN
+F 2 "" H 6650 5000 60  0000 C CNN
+F 3 "" H 6650 5000 60  0000 C CNN
+	1    6650 5000
+	0    -1   -1   0
+$EndComp
+$Comp
+L CONN_1 H3
+U 1 1 53077F2E
+P 6850 5000
+F 0 "H3" V 6950 4975 40  0000 L CNN
+F 1 "CONN_1" H 6850 5055 30  0001 C CNN
+F 2 "" H 6850 5000 60  0000 C CNN
+F 3 "" H 6850 5000 60  0000 C CNN
+	1    6850 5000
+	0    -1   -1   0
+$EndComp
+$Comp
+L CONN_1 H4
+U 1 1 53077F34
+P 7050 5000
+F 0 "H4" V 7150 4975 40  0000 L CNN
+F 1 "CONN_1" H 7050 5055 30  0001 C CNN
+F 2 "" H 7050 5000 60  0000 C CNN
+F 3 "" H 7050 5000 60  0000 C CNN
+	1    7050 5000
+	0    -1   -1   0
+$EndComp
+NoConn ~ 6450 5150
+NoConn ~ 6650 5150
+NoConn ~ 6850 5150
+NoConn ~ 7050 5150
 $EndSCHEMATC
